Commit message: joint_6_m state - fixed

File: abb_irb120_support/urdf/irb120_3_58_macro.xacro (robot description, xacro)
@@ -411,5 +411,5 @@
     </joint>
     <joint name="${prefix}joint_6_m" type="revolute">
-      <origin rpy="0 0 0" xyz="-0.302 0 0"/>
+      <origin rpy="0 -1.0821 0" xyz="-0.302 0 0"/>
       <parent link="${prefix}link_4_m"/>
       <child link="${prefix}link_5_m"/>
